File: amc6821/eagle/av_unit_fan_control/av_unit_fan_ctrl.brd (EAGLE design)
At the start: 68.6 x 53.3 mm, 56 parts, among them U1 AMC6821, U2 AMC6821, U3 AMC6821, U4 AMC6821, X1 DISCDRIVER

Commit message: _
Parts:
- moved C5 1.27 mm to (10.8, 48.9)
- turned FAULT to 90 degrees
Routing:
- net GND: track 73.6 -> 54.1 mm
- net N$11: track 13.3 -> 21.0 mm
- net D13: track 27.0 -> 23.3 mm
- net N$12: track 13.8 -> 11.3 mm
- net D7: track 29.2 -> 27.9 mm
- net ~D11: track 41.9 -> 40.7 mm
- net ~D9: track 34.2 -> 33.1 mm
- net D12: track 39.1 -> 38.1 mm
- net A5-SCL: track 140.2 -> 139.3 mm
- net D2-INT0: track 100.6 -> 99.7 mm
- net ~D5: track 67.8 -> 67.0 mm
- net 5V: track 271.2 -> 270.5 mm
- net D4: track 29.6 -> 29.1 mm
- net A4-SDA: track 130.9 -> 130.4 mm
- net ~D3-INT1: track 74.3 -> 73.8 mm
