File: EAGLE/amc6821-breakout-v2.3.sch (EAGLE design)
At the start: 66 parts, among them J1 Qwiic, J2 Qwiic, J5 KK-254-4KK-254, Q1 2N3904, Q2 2N7002, Q3 310mA/60V/1.6Ω, Q4 310mA/60V/1.6Ω, Q5 NDT3055L, U1 AMC6821-Q1QSOP-16N, U2 SN74LVC2G14DCKR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

Commit message: re-upload of v2.3
Parts:
- removed 5V-FAN: JST-PH-2, VinoRodrigues_Custom_Eagle:JST-PH-2
- removed FD1, FD2, FD3, FD4: FIDUCIALUFIDUCIAL, SparkFun-Aesthetics:FIDUCIALUFIDUCIAL
- removed J7: (no value), SparkFun-Connectors:CONN_02
- removed J8: (no value), SparkFun-Connectors:CONN_01
- removed R8: 10k, SparkFun-Resistors:10KOHM-0603-1/10W-1%
- added D5: 200mA/100V/1V, SparkFun-DiscreteSemi:DIODE-1N4148
- added J11: (no value), SparkFun-Connectors:CONN_01
- added JP0: JUMPER-SMT_3_1-NC_TRACE_SILK, SparkFun-Jumpers:JUMPER-SMT_3_1-NC_TRACE_SILK
- added JP8: (no value), SparkFun-Connectors:CONN_04X2
- added JP9: (no value), SparkFun-Connectors:CONN_03X2NO_SILK
- added R13, R14: 10k, SparkFun-Resistors:10KOHM-0603-1/10W-1%
- added R15: 4.7k, SparkFun-Resistors:4.7KOHM-0603-1/10W-1%
- added U$1: TECSMITH-LOGO, VinoRodrigues_Custom_Eagle:TECSMITH-LOGO
- C7: value 1.0nF -> 1nF; device SparkFun-Capacitors:1.0NF/1000PF-0402_TIGHT-50V-10% -> SparkFun-Capacitors:1.0NF/1000PF-0603-50V-10%
- J1, J2: value Qwiic -> QWIIC_RIGHT_ANGLE; device VinoRodrigues_Custom_Eagle:QWIIC_CONNECTOR -> SparkFun-Connectors:QWIIC_CONNECTORJS-1MM
- J10: value (none) -> 455-1750-1-ND; device SparkFun-Connectors:CONN_021X02_NO_SILK -> SparkFun-Connectors:CONN_03
- J12: device SparkFun-Connectors:CONN_03X2NO_SILK -> SparkFun-Connectors:CONN_01
- J14: device SparkFun-Connectors:CONN_01 -> SparkFun-Connectors:CONN_02
- J6: value (none) -> FAN No2; device SparkFun-Connectors:CONN_02 -> VinoRodrigues_Custom_Eagle:JST-PH-2
- J9: device SparkFun-Connectors:CONN_04PTH -> SparkFun-Connectors:CONN_02
- JP1: value JUMPER-SMT_3_2-NC_TRACE_SILK -> JUMPER-SMT_3_1-NC_TRACE_SILK; device SparkFun-Jumpers:JUMPER-SMT_3_2-NC_TRACE_SILK -> SparkFun-Jumpers:JUMPER-SMT_3_1-NC_TRACE_SILK
- JP3: value JUMPER-SMT_3_1-NC_TRACE_SILK -> JUMPER-SMT_3_2-NC_TRACE_SILK; device SparkFun-Jumpers:JUMPER-SMT_3_1-NC_TRACE_SILK -> SparkFun-Jumpers:JUMPER-SMT_3_2-NC_TRACE_SILK
- JP7: value JUMPER-SMT_3_1-NC_TRACE_SILK -> JUMPER-SMT_2_NC_TRACE_SILK; device SparkFun-Jumpers:JUMPER-SMT_3_1-NC_TRACE_SILK -> SparkFun-Jumpers:JUMPER-SMT_2_NC_TRACE_SILK
- Q2: device SparkFun-DiscreteSemi:MOSFET-NCH-2N7002PW -> VinoRodrigues_Custom_Eagle:2N7002-BSS138
- Q3, Q4: value 310mA/60V/1.6Ω -> 2N7002-BSS138; device SparkFun-DiscreteSemi:MOSFET-NCH-2N7002PW -> VinoRodrigues_Custom_Eagle:2N7002-BSS138
- R1, R10, R11, R12, R2, R9: value 3.3K -> 4.7K
- R3, R4, R5, R6: value 330 -> 1K
- R7: value 1.5k -> 2.2k
Connections:
- removed net !SHDN: J10.1, J10.2
- removed net N$30: JP7.2, U1.PWM-OUT
- removed net SENS: J5.3:TACH, J8.1, R8.1, U1.TACH
- new net N$12: JP5.1, R6.2
- new net N$17: J5.3:TACH, JP9.4, R14.2
- new net N$18: JP9.2, R13.2
- new net PWM: JP4.2, U1.PWM-OUT
- new net TACH: J13.1, R14.1, R15.2, U1.TACH
- new net VDD: D5.C, J5.2:+12VDC, JP9.3
- net !FAN-FAULT: now also J10.1; no longer J9.2
- net !OVR: now also J10.3, U2.2A; no longer J9.4, U2.1A
- net !PWM-OUT: now also JP4.3; no longer JP7.1
- net !SMBALERT: now also J11.1; no longer J9.1
- net !THERM: now also J10.2, U2.1A; no longer J9.3, U2.2A
- net 12V: now also JP9.1, R13.1; no longer J5.2:+12VDC
- net 3V3: now also JP0.1, JP1.1, JP3.2, JP5.2; no longer JP1.2, JP3.1, JP4.1, R6.2, R8.2
- net 5V: now also J6.1, JP9.5, JP9.6; no longer 5V-FAN.1
- net FAN-GND: now also D5.A, JP8.3; no longer J12.4
- net GND: now also JP0.3, JP1.3, JP8.1, R15.1; no longer J12.6, JP3.3, JP4.3
- net GND-5V: now also J6.2, JP8.7; no longer 5V-FAN.2, J14.1
- net GND-PWM: now also JP8.5, Q5.D2; no longer J12.2
- net IN+: now also J14.1, JP6.1; no longer J7.1, JP5.1
- net IN-: now also J14.2, JP7.1; no longer J7.2, JP6.1
- net N$1: now also JP0.2; no longer JP2.2
- net N$2: now also J9.1, JP6.2; no longer J6.1, JP5.2
- net N$3: now also JP3.3; no longer JP1.3
- net N$4: now also JP3.1; no longer JP1.1
- net N$5: now also JP2.2; no longer JP4.2
- net N$6: now also JP1.2; no longer JP3.2
- net N$7: now also J9.2, JP7.2; no longer J6.2, JP6.2
- net OVR: now also U2.2Y; no longer U2.1Y
- net PWM-FAN: now also JP8.2; no longer J12.5
- net PWM-MF: now also JP8.6, JP8.8; no longer J12.1, R7.1
- net PWM-OUT: now also J12.1, JP4.1, JP8.4, R7.1; no longer J12.3, J13.1, JP7.3
- net THERM: now also U2.1Y; no longer U2.2Y
Other:
- note added: "Fan Selection Jumpers"
- note added: "Install 7805 or Pololu 5V Regulator if 5V input is n/a"
- note added: "JP0 = A0 pin; 1-2* = VCC, 2-3 = GND, 0 =NC JP1 = A1 pin; 1-2* = VCC, 2-3 = GND, 0 = NC JP2 = PWM-MODE; 1-2* = xxx, 2-3 = yyy JP3 = I2C Pullups; 1-2-3* = enabled, 0 = cut JP4 = PWM-Mode (Hard); 1-2* = normal, 2-3 = inverted, 0 = diabled (do not use) JP5 = Power LED; 1-2* = enabled, 0 = off JP6, JP7 = Remote Temp Sensor; 1-2* = enabled, 0 = disconnected (reconnect via J9)"
- note added: "JP8 = Fan Selection #1357 Row -> Grounding 1-3 = 12VDC 4-Wire fan 3-5 = 12VDC 3-Wire fan 5-7 = 5VDC 2- or 3-Wire fan #2468 Row -> PWM Signal 2-4 = PWM to FAN pin 4 4-6 = PWM to (N-)MOSFET (for 3-Wire fan) 6-8 = PWM off (for 2-Wire fan) JP9 = Voltage Divider short-circuit #135 Row -> FAN POWER (VDD) 1-3 = 12VDC supply 3-5 = 5VDC Supply #246 Row -> SENS Pull-UP Supply 2-4 = 12VDC supply (adds 10KOh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"
- note added: "Jumper Settings"
- note added: "PWM MOSFET (for 3- & 2- Wire Fans)"
- note added: "Remote Temp. Sensor (Cutout)"
- note added: "Signal Inversion"
- note added: "Status LEDs"
- note removed: "Optional Temp. Sensor"
- note removed: "PWM"
- moved on the sheet: C1, C2, C3, C4, C5, C6, C7, D1, D2, D3, D4, J13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
