File: EAGLE/amc6821-breakout-v2.3.brd (EAGLE design)
At the start: 45.7 x 45.8 mm, 68 parts, among them J1 QWIIC_RIGHT_ANGLE, J10 455-1750-1-ND, J2 QWIIC_RIGHT_ANGLE, J5 KK-254-4KK-254, J6 FAN No2, Q1 2N3904, Q2 2N7002, Q5 NDT3055L, U1 AMC6821-Q1QSOP-16N, U2 SN74LVC2G14DCKR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

Commit message: clean up of v2.3
Routing:
- net !PWM-OUT: track 15.4 -> 14.9 mm, vias 2 -> 1
Changed lines of the file:
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@@
 <wire x1="29.8704" y1="6.5786" x2="29.8704" y2="5.6896" width="0.3556" layer="1"/>
 <wire x1="29.8704" y1="5.6896" x2="30.48" y2="5.08" width="0.3556" layer="1"/>
-<wire x1="30.48" y1="5.08" x2="27.686" y2="5.08" width="0.3556" layer="16"/>
-<wire x1="27.686" y1="5.08" x2="27.051" y2="4.445" width="0.3556" layer="16"/>
-<via x="27.051" y="4.445" extent="1-16" drill="0.35"/>
 <contactref element="JP4" pad="3"/>
 <wire x1="19.05" y1="9.1186" x2="19.3294" y2="9.1186" width="0.3556" layer="16"/>
 <wire x1="22.225" y1="6.223" x2="19.3294" y2="9.1186" width="0.3556" layer="16"/>
-<wire x1="26.289" y1="4.445" x2="24.511" y2="6.223" width="0.3556" layer="16"/>
-<wire x1="26.289" y1="4.445" x2="27.051" y2="4.445" width="0.3556" layer="16"/>
+<wire x1="25.654" y1="5.08" x2="24.511" y2="6.223" width="0.3556" layer="16"/>
+<wire x1="25.654" y1="5.08" x2="30.48" y2="5.08" width="0.3556" layer="16"/>
 <wire x1="22.225" y1="6.223" x2="24.511" y2="6.223" width="0.3556" layer="16"/>
 </signal>
