File: EAGLE/amc6821-breakout-v3.0.brd (EAGLE design)
At the start: 34.3 x 25.4 mm, 37 parts, among them J8 QWIIC_RIGHT_ANGLE, J9 QWIIC_RIGHT_ANGLE, Q1 2N3904, U1 AMC6821-Q1QSOP-16N, U3 AP2112K-3.3

Commit message: wip
Parts:
- Q1: value 2N3904 -> MMBT3904 SOT-23
Changed lines of the file:
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@@
 <drawing>
 <settings>
-<setting alwaysvectorfont="yes"/>
+<setting alwaysvectorfont="no"/>
 <setting verticaltext="up"/>
 </settings>
@@
 <element name="LOGO1" library="SparkFun-Aesthetics" package="OSHW-LOGO-S" value="OSHW-LOGOS" x="12.7" y="17.907" smashed="yes" rot="MR0"/>
 <element name="LOGO2" library="SparkFun-Aesthetics" package="QWIIC_6MM" value="QWIIC_LOGO_6MM" x="3.302" y="12.7" smashed="yes" rot="R90"/>
-<element name="Q1" library="SparkFun-DiscreteSemi" package="SOT23-3" value="2N3904" x="30.48" y="7.62" smashed="yes" rot="R180">
+<element name="Q1" library="SparkFun-DiscreteSemi" package="SOT23-3" value="MMBT3904 SOT-23" x="30.48" y="7.62" smashed="yes" rot="R180">
 <attribute name="NAME" x="30.48" y="7.366" size="0.6096" layer="25" font="vector" ratio="20" align="bottom-center"/>
 <attribute name="PROD_ID" value="TRANS-09116" x="-21.59" y="86.36" size="1.778" layer="27" rot="R180" display="off"/>
