File: EAGLE/fan-host-board-v1.1-(WIP).sch (EAGLE design)
At the start: 36 parts, among them J8 QWIIC_RIGHT_ANGLE, J9 QWIIC_RIGHT_ANGLE, Q1 MMBT3904 SOT-23, U1 AMC6821-Q1QSOP-16N, U3 AP2112K-3.3

Commit message: wip
Parts:
- removed C3: 0.1uF, SparkFun-Capacitors:0.1UF-0603-25V-5%
- removed C4: 1nF, SparkFun-Capacitors:1.0NF/1000PF-0603-50V-10%
- removed D4: GREEN, SparkFun-LED:LED-GREEN0603
- removed J8, J9: QWIIC_RIGHT_ANGLE, VinoRodrigues_Custom_Eagle:QWIIC_CONNECTOR_GNDJS-1MM
- removed JP0: JUMPER-SMT_3_1-NC_TRACE_SILK, SparkFun-Jumpers:JUMPER-SMT_3_1-NC_TRACE_SILK
- removed LOGO2: QWIIC_LOGO_6MM, SparkFun-Aesthetics:QWIIC_LOGO_6MM
- removed Q1: MMBT3904 SOT-23, SparkFun-DiscreteSemi:TRANS_NPN-MMBTA42
- removed R5, R6: 2.2k, SparkFun-Resistors:2.2KOHM-0603-1/10W-1%
- removed R7: 1K, SparkFun-Resistors:RESISTOR0805
- removed U1: AMC6821-Q1QSOP-16N, VinoRodrigues_Custom_Eagle:AMC6821-Q1QSOP-16N
- removed U3: AP2112K-3.3, microbuilder:VREG_SOT23-5
- added 12V-FAN: KK-254-4KK-254, VinoRodrigues_Custom_Eagle:KK-254-4KK-254
- added 5V-FAN: JST-PH-2, VinoRodrigues_Custom_Eagle:JST-PH-2
- added CN1: (no value), adafruit:JST_2PIN-THM
- added D1: 200mA/100V, SparkFun-DiscreteSemi:DIODE-1N4148
- added D2: 1A/40V, SparkFun-DiscreteSemi:DIODE-SCHOTTKY-SS14
- added J1: (no value), SparkFun-Connectors:CONN_05
- added J2: (no value), SparkFun-Connectors:CONN_06SILK_FEMALE_PTH
- added JP5: Cut when MOSFET in use, SparkFun-Jumpers:JUMPER-SMT_2_NC_TRACE_NO-SILK
- added U$11, U$2, U$3, U$6: MOUNTINGHOLE2.5, microbuilder:MOUNTINGHOLE2.5
- added U$14: NDT3055L, VinoRodrigues_Custom_Eagle:NDT3055L
- added VREG: TRACOPOWER-TSR-1, VinoRodrigues_Custom_Eagle:TRACOPOWER-TSR-1
- C1: value 10uF -> 0.33µF; device SparkFun-Capacitors:10UF-0603-6.3V-20% -> SparkFun-Capacitors:0.33UF/330NF-0805-50V-10%
- C2: value 10uF -> 0.1uF; device SparkFun-Capacitors:10UF-0603-6.3V-20% -> SparkFun-Capacitors:0.1UF-0603-25V-5%
- J3: device SparkFun-Connectors:CONN_05 -> SparkFun-Connectors:CONN_04PTH
- J5: device SparkFun-Connectors:CONN_01 -> SparkFun-Connectors:CONN_02PTH3
- J6: device SparkFun-Connectors:CONN_01 -> SparkFun-Connectors:CONN_04SCREW
- J7: device VinoRodrigues_Custom_Eagle:CONN_02 -> SparkFun-Connectors:CONN_021X02_NO_SILK
- JP1: value JUMPER-SMT_3_1-NC_TRACE_SILK -> JUMPER-VSELECT
- JP2: value JUMPER-SMT_3_1-NC_TRACE_SILK -> JUMPER-5V; device SparkFun-Jumpers:JUMPER-SMT_3_1-NC_TRACE_SILK -> VinoRodrigues_Custom_Eagle:JUMPER-SMT_2_NO_NO_SILK
- JP3: value JUMPER-SMT_3_2-NC_TRACE_SILK -> JUMPER-12V-a; device SparkFun-Jumpers:JUMPER-SMT_3_2-NC_TRACE_SILK -> SparkFun-Jumpers:JUMPER-SMT_2_NC_TRACE_SILK
- JP4: value JUMPER-SMT_2_NC_TRACE_SILK -> JUMPER-12V-b
- R1: value 2.2k -> 10k for MOSFET, 2k for PWM fan
- R2, R3: value 2.2k -> 10k; device SparkFun-Resistors:2.2KOHM-0603-1/10W-1% -> SparkFun-Resistors:10KOHM-0603-1/10W-1%
- R4: value 2.2k -> 4.7k; device SparkFun-Resistors:2.2KOHM-0603-1/10W-1% -> SparkFun-Resistors:4.7KOHM-0603-1/10W-1%
Connections:
- removed net !OVR: J5.1, R4.1, U1.!OVR
- removed net !THERM: J6.1, R5.1, U1.!THERM
- removed net N$1: JP0.2, U1.A0
- removed net N$12: JP4.1, R7.2
- removed net N$3: JP3.3, R2.1
- removed net N$8: D4.A, R7.1
- new net 12V: 12V-FAN.2:+12VDC, C1.1, D1.C, J6.1, JP1.3, VREG.IN
- new net GND-3: 12V-FAN.1:GND, 5V-FAN.2, D1.A, D2.A, JP5.2, U$14.D, U$14.D2
- new net SHDN: J7.1, J7.2
- new net TACH/SENS: 12V-FAN.3:TACH, JP2.2, R2.2, R3.1
- net !FAN-FAULT: now also J1.5; no longer J3.5, R6.1, U1.!FAN-FAULT
- net !SMBALERT: now also J2.6; no longer J4.6, R3.1, U1.!SMBALERT
- net 3V3: now also J2.2, R1.2; no longer C2.1, C3.2, J8.2, J9.2, JP0.1, JP1.1, JP2.1, JP3.2, JP4.2, R3.2, R4.2, R5.2, R6.2, U1.VDD, U3.OUT
- net 5V: now also 5V-FAN.1, C2.1, D2.C, J2.1, J6.4, JP1.1, VREG.OUT; no longer C1.1, U3.EN, U3.IN
- net GND: now also J2.3, J6.2, J6.3, JP5.1, R4.2, U$14.S, VREG.GND; no longer C3.1, D4.C, J8.1, J8.NC1, J8.NC2, J9.1, J9.NC1, J9.NC2, JP0.3, JP1.3, JP2.3, U1.GND, U3.GND
- net IN+: now also CN1.2, J1.1, J5.1; no longer C4.2, J7.2, Q1.B, Q1.C, U1.IN+
- net IN-: now also CN1.1, J1.2, J5.2; no longer C4.1, J7.1, Q1.E, U1.IN-
- net N$4: now also JP1.2, R2.1; no longer JP3.1, R1.1
- net N$5: now also JP3.2, R3.2; no longer JP2.2, U1.!PWM-MODE
- net N$6: now also JP4.2, R4.1; no longer JP1.2, U1.A1
- net PWM: now also 12V-FAN.4:PWM, J1.3, R1.1, U$14.G; no longer U1.PWM-OUT
- net SCL: now also J2.4; no longer J8.4, J9.4, R1.2, U1.SCLK
- net SDA: now also J2.5; no longer J8.3, J9.3, R2.2, U1.SDA
- net TACH: now also J1.4, JP2.1, JP3.1, JP4.1; no longer U1.TACH
Other:
- note added: "(If 5V not present)"
- note added: "DO NOT INCLUDE when using 5V diode"
- note added: "Fan(s)"
- note added: "Install 5V Voltage Regulator (for max Amps) * Pololu D24V3F5 -> 300mA (no fan recm.) * Pololu D25V6F4 -> 500mA * TracoPower TSR-1-2450 -> 1A * LM7805 -> 1.5A"
- note added: "Not used. Provided in case Pololu 4-pin module used."
- note added: "Optional"
- note added: "Optional 12V to 5V"
- note added: "Power Input Header"
- note removed: "5V to 3.3V"
- note removed: "AMC6821 IC"
- note removed: "I2C / Qwiic Bus"
- note removed: "Pin Pull-ups"
- note removed: "Power LED (Optional)"
- note removed: "Remote Temp. Sensor (Cutout)"
- moved on the sheet: C1, C2, J4, J7, JP1, JP4, R1, R2, R3, R4
