File: EAGLE/old/amc6821-breakout-v2.2.brd (EAGLE design)
At the start: 45.7 x 38.1 mm, 67 parts, among them J1 Qwiic, J2 Qwiic, J5 KK-254-4KK-254, Q1 2N3904, Q2 2N7002, Q3 310mA/60V/1.6Ω, Q4 310mA/60V/1.6Ω, Q5 NDT3055L, U1 AMC6821-Q1QSOP-16N, U2 SN74LVC2G14DCKR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

Commit message: re-upload of v2.3
Parts:
- removed 5V-FAN: JST-PH-2, VinoRodrigues_Custom_Eagle:JST-PH2
- added J11: (no value), SparkFun-Connectors:1X01
- added J15: (no value), SparkFun-Connectors:1X02_NO_SILK
- added JP0: JUMPER-SMT_3_1-NC_TRACE_SILK, SparkFun-Jumpers:SMT-JUMPER_3_1-NC_TRACE_SILK
- C7: value 1.0nF -> 1nF; device SparkFun-Capacitors:0402-TIGHT -> SparkFun-Capacitors:0603
- J1, J2: value Qwiic -> QWIIC_RIGHT_ANGLE; device VinoRodrigues_Custom_Eagle:JST04_1MM_VERT -> SparkFun-Connectors:JST04_1MM_RA
- J10: value (none) -> 455-1750-1-ND; device SparkFun-Connectors:1X02_NO_SILK -> SparkFun-Connectors:1X03
- J12: device SparkFun-Connectors:2X3-NS -> SparkFun-Connectors:1X01
- J14: device SparkFun-Connectors:1X01 -> SparkFun-Connectors:1X02
- J6: value (none) -> JST-PH-2; device SparkFun-Connectors:1X02 -> VinoRodrigues_Custom_Eagle:JST-PH2
- J7: device SparkFun-Connectors:1X02 -> SparkFun-Connectors:2X3-NS
- J9: device SparkFun-Connectors:1X04 -> SparkFun-Connectors:1X02
- JP1: value JUMPER-SMT_3_2-NC_TRACE_SILK -> JUMPER-SMT_3_1-NC_TRACE_SILK; device SparkFun-Jumpers:SMT-JUMPER_3_2-NC_TRACE_SILK -> SparkFun-Jumpers:SMT-JUMPER_3_1-NC_TRACE_SILK
- JP3: value JUMPER-SMT_3_1-NC_TRACE_SILK -> JUMPER-SMT_3_2-NC_TRACE_SILK; device SparkFun-Jumpers:SMT-JUMPER_3_1-NC_TRACE_SILK -> SparkFun-Jumpers:SMT-JUMPER_3_2-NC_TRACE_SILK
- JP7: value JUMPER-SMT_3_1-NC_TRACE_SILK -> JUMPER-SMT_2_NC_TRACE_SILK; device SparkFun-Jumpers:SMT-JUMPER_3_1-NC_TRACE_SILK -> SparkFun-Jumpers:SMT-JUMPER_2_NC_TRACE_SILK
- Q2: device SparkFun-DiscreteSemi:SOT323 -> VinoRodrigues_Custom_Eagle:SOT23-3
- Q3, Q4: value 310mA/60V/1.6Ω -> (none); device SparkFun-DiscreteSemi:SOT323 -> VinoRodrigues_Custom_Eagle:SOT23-3
- R1, R10, R11, R12, R2, R9: value 3.3K -> 4.7K
- R3, R4, R5, R6: value 330 -> 1K
- moved J10 42.7 mm to (12.7, 1.91), flipped to the top, turned to 180 degrees
- moved J9 27.9 mm to (1.27, 26.0), turned to 0 degrees
- moved J12 21.7 mm to (27.9, 1.91)
- moved JP7 20.8 mm to (21.6, 33.7), turned to 270 degrees
- moved J8 20.2 mm to (9.53, 20.3), turned to 90 degrees
- moved JP4 19.2 mm to (19.7, 13.0), turned to 180 degrees
- moved JP1 13.7 mm to (34.3, 19.1), turned to 90 degrees
- moved JP3 13.7 mm to (29.2, 6.35), turned to 0 degrees
- moved J7 13.4 mm to (14.6, 19.1)
- moved JP2 12.7 mm to (34.3, 25.4)
- moved J13 10.2 mm to (17.8, 1.91)
- moved J14 8.26 mm to (1.27, 20.3), turned to 0 degrees
- moved J6 7.65 mm to (8.89, 26.7), turned to 90 degrees
- moved LOGO5 0.90 mm to (38.4, 9.27)
- moved J1 0.81 mm to (40.1, 9.53), turned to 90 degrees
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Connections:
- new net N$12: JP7.1, R6.2
- net !FAN-FAULT: now also J10.1; no longer J9.2
- net !OVR: now also J10.3; no longer J9.4
- net !PWM-OUT: now also JP4.1; no longer JP7.1
- net !SHDN: now also J15.1, J15.2; no longer J10.1, J10.2
- net !SMBALERT: now also J12.1; no longer J9.1
- net !THERM: now also J10.2; no longer J9.3
- net 3V3: now also JP0.1, JP1.1, JP3.2, JP7.2; no longer JP1.2, JP3.1, JP4.1, R6.2
- net 5V: now also J6.1; no longer 5V-FAN.1
- net FAN-GND: now also J7.4; no longer J12.4
- net GND: now also J7.6, JP0.3, JP1.3; no longer J12.6, JP3.3, JP4.3
- net GND-5V: now also J6.2, J8.1; no longer 5V-FAN.2, J14.1
- net GND-PWM: now also J7.2; no longer J12.2
- net IN+: now also J14.1; no longer J7.1
- net IN-: now also J14.2; no longer J7.2
- net N$1: now also JP0.2; no longer JP2.2
- net N$2: now also J9.1; no longer J6.1
- net N$3: now also JP3.3; no longer JP1.3
- net N$30: now also JP4.2; no longer JP7.2
- net N$4: now also JP3.1; no longer JP1.1
- net N$5: now also JP2.2; no longer JP4.2
- net N$6: now also JP1.2; no longer JP3.2
- net N$7: now also J9.2; no longer J6.2
- net PWM-FAN: now also J7.5; no longer J12.5
- net PWM-MF: now also J7.1; no longer J12.1
- net PWM-OUT: now also J11.1, J7.3, JP4.3; no longer J12.3, J13.1, JP7.3
- net SENS: now also J13.1; no longer J8.1
Routing:
- net PWM-OUT: track 41.9 -> 48.3 mm
- net !SMBALERT: track 18.7 -> 24.7 mm
- net SCL: track 39.0 -> 44.7 mm, vias 2 -> 3
- net 3V3: track 162.3 -> 166.5 mm, vias 12 -> 13
- net N$12: track 0.00 -> 3.90 mm, vias 0 -> 1
- net GND: track 0.00 -> 3.00 mm, vias 14 -> 20
- net N$7: track 5.71 -> 7.82 mm
- net N$2: track 8.05 -> 10.2 mm
- net SDA: track 38.8 -> 36.7 mm, vias 3 -> 1
- net !THERM: track 27.3 -> 27.9 mm
- net GND-PWM: track 14.8 -> 14.3 mm
Other:
- board text added: "!F"
- board text added: "!THRM"
- board text added: "AMC6821 Breakout Board | Rel 2.2 (c) 2020 Vino Rodrigues http://tecsmith.com.au"
- board text added: "PW"
- board text added: "PWM- MOSFET"
- board text added: "SCL SDA 3V3 GND"
- board text added: "TCH"
- board text removed: "!FAULT"
- board text removed: "AMC6821 Breakout Board | Rel 2.0 (c) 2020 Vino Rodrigues http://tecsmith.com.au"
- board text removed: "GND 3V3 SDA SCL"
- board text removed: "PWM-MOSFET"
