File: EAGLE/old/amc6821-breakout-v2.2.sch (EAGLE design)
At the start: 24 parts, among them U1 ESP8266_ESP-01, U2 REG1117-3.3

Commit message: re-upload of v2.3
Parts:
- removed 3V3: (no value), SparkFun-Connectors:CONN_01PTH_NO_SILK_YES_STOP
- removed S1: RESET, SparkFun-Switches:MOMENTARY-SWITCH-SPST-2-SMD-5.2MM
- added C4, C5: 10uF, SparkFun-Capacitors:10UF-0603-6.3V-20%
- added C6: 0.1uF, SparkFun-Capacitors:0.1UF-0603-25V-5%
- added C7: 1nF, SparkFun-Capacitors:1.0NF/1000PF-0603-50V-10%
- added D2, D3: RED, SparkFun-LED:LED-RED0603
- added D4: GREEN, SparkFun-LED:LED-GREEN0603
- added FD1, FD2, FD3, FD4: FIDUCIALUFIDUCIAL, SparkFun-Aesthetics:FIDUCIALUFIDUCIAL
- added H3, H4, H5, H6: STAND-OFF, SparkFun-Hardware:STAND-OFF
- added J10: 455-1750-1-ND, SparkFun-Connectors:CONN_03
- added J11, J12, J13, J8: (no value), SparkFun-Connectors:CONN_01
- added J14, J9: (no value), SparkFun-Connectors:CONN_02
- added J15: (no value), SparkFun-Connectors:CONN_021X02_NO_SILK
- added J5: KK-254-4KK-254, VinoRodrigues_Custom_Eagle:KK-254-4KK-254
- added JP0, JP2, JP4: JUMPER-SMT_3_1-NC_TRACE_SILK, SparkFun-Jumpers:JUMPER-SMT_3_1-NC_TRACE_SILK
- added JP3: JUMPER-SMT_3_2-NC_TRACE_SILK, SparkFun-Jumpers:JUMPER-SMT_3_2-NC_TRACE_SILK
- added JP5, JP6, JP7: JUMPER-SMT_2_NC_TRACE_SILK, SparkFun-Jumpers:JUMPER-SMT_2_NC_TRACE_SILK
- added Q1: 2N3904, SparkFun-DiscreteSemi:TRANS_NPN-MMBTA42
- added Q2: 2N7002, VinoRodrigues_Custom_Eagle:2N7002-BSS138
- added Q3, Q4: 2N7002-BSS138, VinoRodrigues_Custom_Eagle:2N7002-BSS138
- added Q5: NDT3055L, VinoRodrigues_Custom_Eagle:NDT3055L
- added R10, R11, R12, R9: 4.7K, SparkFun-Resistors:RESISTOR0805
- added R6: 1K, SparkFun-Resistors:RESISTOR0805
- added R7: 1.5k, SparkFun-Resistors:1.5KOHM-0603-1/10W-1%
- added R8: 10k, SparkFun-Resistors:10KOHM-0603-1/10W-1%
- added U3: SN74LVC2G14DCKR, VinoRodrigues_Custom_Eagle:SN74LVC2G14DCKR
- added U4: LD1117-33, SparkFun-IC-Power:V_REG_LD1117VXXLD1117-SMD
- added U5: 7805TV, linear:7805TV
- C1: value 10uF -> 0.33µF; device SparkFun-Capacitors:10UF-POLAR-EIA3216-16V-10%(TANT) -> SparkFun-Capacitors:0.33UF/330NF-0805-50V-10%
- C2: value 22uF -> 0.1uF; device SparkFun-Capacitors:22UF-0805-6.3V-20% -> SparkFun-Capacitors:0.1UF-0603-25V-5%
- C3: value 0.1uF -> 10uF; device SparkFun-Capacitors:0.1UF-0603-25V-5% -> SparkFun-Capacitors:10UF-0603-6.3V-20%
- D1: value BLUE -> RED; device SparkFun-LED:LED-BLUE0603 -> SparkFun-LED:LED-RED0603
- J1: value (none) -> QWIIC_RIGHT_ANGLE; device VinoRodrigues_Custom_Eagle:QWIIC_CONNECTORJST04_1MM_RA_GND -> SparkFun-Connectors:QWIIC_CONNECTORJS-1MM
- J2: value (none) -> QWIIC_RIGHT_ANGLE; device SparkFun-Connectors:I2C_STANDARD -> SparkFun-Connectors:QWIIC_CONNECTORJS-1MM
- J3: device SparkFun-Connectors:6_PIN_SERIAL_TARGETSILK -> SparkFun-Connectors:I2C_STANDARD
- J4: device SparkFun-Connectors:CONN_02 -> SparkFun-Connectors:CONN_04SCREW
- J6: value (none) -> JST-PH-2; device SparkFun-Connectors:CONN_021X02_NO_SILK -> VinoRodrigues_Custom_Eagle:JST-PH-2
- J7: device VinoRodrigues_Custom_Eagle:USB_MICRO-B_FEMALE-SMT -> SparkFun-Connectors:CONN_03X2NO_SILK
- JP1: value JUMPER-SMT_3_2-NC_TRACE_SILK -> JUMPER-SMT_3_1-NC_TRACE_SILK; device SparkFun-Jumpers:JUMPER-SMT_3_2-NC_TRACE_SILK -> SparkFun-Jumpers:JUMPER-SMT_3_1-NC_TRACE_SILK
- R1, R2: value 3.3K -> 4.7K
- R3, R4: value 3.3K -> 1K
- R5: value 330 -> 1K; device SparkFun-Resistors:330OHM-0603-1/10W-1% -> SparkFun-Resistors:RESISTOR0805
- U1: value ESP8266_ESP-01 -> AMC6821-Q1QSOP-16N; device VinoRodrigues_Custom_Eagle:ESP8266_ESP-01 -> VinoRodrigues_Custom_Eagle:AMC6821-Q1QSOP-16N
- U2: value REG1117-3.3 -> SN74LVC2G14DCKR; device Texas Instruments_By_element14_Batch_1:REG1117-3.3 -> VinoRodrigues_Custom_Eagle:SN74LVC2G14DCKR
Connections:
- removed net CTS: J3.CTS
- removed net DTR: J3.DTR
- removed net RXI: J3.TXO, J6.1, U1.RXD
- removed net TXO: J3.RXI, J6.2, U1.TXD
- removed net VCC: 3V3.1, C2.1, C3.1, J1.2, J2.2, J3.VCC, JP1.2, R1.2, R2.2, R5.1, U1.VCC, U2.VOUT, U2.VOUT_2
- new net !FAN-FAULT: J10.1, R11.1, U1.!FAN-FAULT, U3.1A
- new net !OVR: J10.3, R9.1, U1.!OVR, U2.1A
- new net !PWM-OUT: JP4.1, U3.2A
- new net !SHDN: J15.1, J15.2
- new net !SMBALERT: J12.1, R12.1, U1.!SMBALERT
- new net !THERM: J10.2, R10.1, U1.!THERM, U2.2A
- new net 12V: C1.1, J4.1, J5.2:+12VDC, U5.VI
- new net 3V3: C3.1, C5.1, C6.1, J1.2, J2.2, J3.2, JP0.1, JP1.1, JP2.1, JP3.2, JP7.2, R10.2, R11.2, R12.2, R3.2, R4.2, R5.1, R7.2, R8.2, R9.2, U1.VDD, U2.VCC, U3.VCC, U4.OUT
- new net FAN-FAULT: Q4.G, U3.1Y
- new net FAN-GND: J5.1:GND, J7.4
- new net GND-5V: J6.2, J8.1
- new net GND-PWM: J7.2, Q5.D
- new net IN+: J14.1, JP5.1, U1.IN+
- new net IN-: J14.2, JP6.1, U1.IN-
- new net N$1: JP0.2, U1.A0
- new net N$10: D3.C, Q4.D
- new net N$11: D1.A, R3.1
- new net N$12: JP7.1, R6.2
- new net N$14: D1.C, Q2.D
- new net N$15: D2.C, Q3.D
- new net N$16: D2.A, R4.1
- new net N$2: C7.2, J9.1, JP5.2, Q1.B, Q1.C
- new net N$30: JP4.2, U1.PWM-OUT
- new net N$8: D4.A, R6.1
- new net N$9: D3.A, R5.2
- new net OVR: Q2.G, U2.1Y
- new net PWM-FAN: J5.4:PWM, J7.5
- new net PWM-MF: J7.1, Q5.G, R7.1
- new net PWM-OUT: J11.1, J7.3, JP4.3, U3.2Y
- new net SENS: J13.1, J5.3:TACH, R8.1, U1.TACH
- new net THERM: Q3.G, U2.2Y
- net 5V: now also C2.1, C4.1, J4.4, J6.1, U4.IN, U5.VO; no longer C1.+, J7.VBUS, U2.VIN
- net GND: now also C1.2, C4.2, C5.2, C6.2, D4.C, J3.1, J4.2, J4.3, J7.6, JP0.3, JP1.3, JP2.3, Q2.S, Q3.S, Q4.S, Q5.S, U2.GND, U3.GND, U4.GND, U5.GND; no longer C1.-, D1.C, J3.GND, J4.1, J7.GND, S1.3, S1.4, U2.GROUND
- net N$3: now also JP3.3, R1.1; no longer R2.1, S1.1, S1.2, U1.RST
- net N$4: now also JP3.1, R2.1; no longer D1.A, R5.2
- net N$5: now also JP2.2, U1.!PWM-MODE; no longer R1.1, U1.CH_PD
- net N$6: now also JP1.2, U1.A1; no longer JP1.3, R4.2
- net N$7: now also C7.1, J9.2, JP6.2, Q1.E; no longer JP1.1, R3.2
- net SCL: now also J3.4, R2.2, U1.SCLK; no longer R4.1, U1.GPIO2
- net SDA: now also J3.3, R1.2, U1.SDA; no longer J4.2, R3.1, U1.GPIO0
Other:
- note added: "5V to 3.3V"
- note added: "AMC6821 Breakout"
- note added: "AMC6821 IC"
- note added: "Fan(s)"
- note added: "Optional 12V to 5V"
- note added: "Optional Temp. Sensor"
- note added: "PWM"
- note added: "Power"
- note removed: "ESP-01(S) Development Board"
- note removed: "Power Supply"
- note removed: "Programing Header"
- moved on the sheet: C2, C3, D1, J2, J6, R1, R2, R3, R4, R5
